File: noname.kicad_pcb (KiCad board)
At the start: 2 copper layers, 83 parts, among them SW1 Rotary_Encoder_Switch, U1 ProMicro

Commit message: Pm placed edges defined
Parts:
- MX1, MX12: footprint MX_Only:MXOnly-1.5U-NoLED -> MX_Alps_Hybrid:MX-1.5U-NoLED
- MX10, MX11, MX14, MX15, MX16, MX17, MX18, MX19, MX2, MX20, MX21, MX22, MX23, MX26, MX27, MX28, MX29, MX3, MX30, MX31, MX32, MX33, MX34, MX36, MX37, MX39, MX4, MX40, MX5, MX6, MX7, MX8, MX9: footprint MX_Only:MXOnly-1U-NoLED -> MX_Alps_Hybrid:MX-1U-NoLED
- MX13: footprint MX_Only:MXOnly-1.75U-NoLED -> MX_Alps_Hybrid:MX-1.75U-NoLED
- MX24, MX25: footprint MX_Only:MXOnly-2.25U-NoLED -> MX_Alps_Hybrid:MX-2.25U-NoLED
- MX35: footprint MX_Only:MXOnly-2.75U-NoLED -> MX_Alps_Hybrid:MX-2.75U-NoLED
- MX38: footprint MX_Only:MXOnly-7U-NoLED -> MX_Alps_Hybrid:MX-10U-ReversedStabilizers-NoLED
- U1: moved to B.Cu
- moved D41 262.8 mm to (262.7, 138.1), turned to 90 degrees
- moved D14 258.5 mm to (41.3, 100.0), turned to 90 degrees
- moved D40 238.2 mm to (243.7, 138.1), turned to 90 degrees
- moved D28 233.4 mm to (96.0, 119.1), turned to 90 degrees
- moved D29 228.3 mm to (115.1, 119.1), turned to 90 degrees
- moved D15 223.9 mm to (67.5, 100.0), turned to 90 degrees
- moved U1 218.8 mm to (37.1, 96.4)
- moved D16 215.5 mm to (86.5, 100.0), turned to 90 degrees
- moved D18 211.9 mm to (124.6, 100.0), turned to 90 degrees
- moved D33 211.3 mm to (191.3, 119.1), turned to 90 degrees
- moved D17 208.5 mm to (105.6, 100.0), turned to 90 degrees
- moved D5 203.7 mm to (119.9, 81.0), turned to 90 degrees
- moved D32 187.8 mm to (172.2, 119.1), turned to 90 degrees
- moved D36 183.7 mm to (232.6, 119.1), turned to 90 degrees
- moved D3 175.9 mm to (81.8, 81.0), turned to 90 degrees
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Connections:
- SW1 pad A: ENC1 -> (no net)
- SW1 pad B: ENC0 -> (no net)
- SW1 pad C: GND -> (no net)
- U1 pad 1: Net-(U1-Pad1) -> (no net)
- U1 pad 10: Net-(U1-Pad10) -> (no net)
- U1 pad 11: Net-(U1-Pad11) -> (no net)
- U1 pad 12: Net-(U1-Pad12) -> (no net)
- U1 pad 13: Net-(U1-Pad13) -> (no net)
- U1 pad 14: Net-(U1-Pad14) -> (no net)
- U1 pad 15: Net-(U1-Pad15) -> (no net)
- U1 pad 16: Net-(U1-Pad16) -> (no net)
- U1 pad 17: Net-(U1-Pad17) -> (no net)
- U1 pad 18: Net-(U1-Pad18) -> (no net)
- U1 pad 19: Net-(U1-Pad19) -> (no net)
- U1 pad 2: Net-(U1-Pad2) -> (no net)
- U1 pad 20: Net-(U1-Pad20) -> (no net)
- U1 pad 21: Net-(U1-Pad21) -> (no net)
- U1 pad 22: Net-(U1-Pad22) -> (no net)
- U1 pad 23: Net-(U1-Pad23) -> (no net)
- U1 pad 24: Net-(U1-Pad24) -> (no net)
- U1 pad 3: Net-(U1-Pad3) -> (no net)
- U1 pad 4: Net-(U1-Pad4) -> (no net)
- U1 pad 5: Net-(U1-Pad5) -> (no net)
- U1 pad 6: Net-(U1-Pad6) -> (no net)
- U1 pad 7: Net-(U1-Pad7) -> (no net)
- U1 pad 8: Net-(U1-Pad8) -> (no net)
- U1 pad 9: Net-(U1-Pad9) -> (no net)
Other:
- board outline added: 266.7 x 76.2 mm
