File: Full-Bar-rot.kicad_pcb (KiCad board)
At the start: 2 copper layers, 266.7 x 76.2 mm, 84 parts, among them SW1 Rotary_Encoder_Switch, U1 ProMicro

Commit message: traces ran
Parts:
- removed MX41: MX-NoLED, MX_Alps_Hybrid:MX-1U-NoLED
Routing:
- net COL12: track 314.0 -> 248.1 mm, vias 1 -> 0
- net Net-(D13-Pad2): track 12.9 -> 0.00 mm
- net GND: track 266.4 -> 267.1 mm
Changed lines of the file:
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@@
     (thickness 1.6)
     (drawings 8)
-    (tracks 379)
+    (tracks 361)
     (zones 0)
-    (modules 84)
+    (modules 83)
     (nets 60)
   )
@@
     (add_net COL8)
     (add_net COL9)
-    (add_net ENC0)
-    (add_net ENC1)
     (add_net "Net-(D1-Pad2)")
     (add_net "Net-(D10-Pad2)")
@@
     (add_net "Net-(D8-Pad2)")
     (add_net "Net-(D9-Pad2)")
-    (add_net "Net-(U1-Pad21)")
-    (add_net "Net-(U1-Pad22)")
     (add_net ROW0)
     (add_net ROW1)
@@
     (add_net GND)
   )
-  (module MX_Alps_Hybrid:MX-1U-NoLED (layer F.Cu)
-    (at 272.25625 76.99375)
-    (fp_text reference MX41 (at 0 3.175) (layer Dwgs.User)
-      (effects (font (size 1 1) (thickness 0.15)))
-    )
-    (fp_text value MX-NoLED (at 0 -7.9375) (layer Dwgs.User)
-      (effects (font (size 1 1) (thickness 0.15)))
-    )
-    (fp_line (start -9.525 9.525) (end -9.525 -9.525) (layer Dwgs.User) (width 0.15))
-    (fp_line (start 9.525 9.525) (end -9.525 9.525) (layer Dwgs.User) (width 0.15))
-    (fp_line (start 9.525 -9.525) (end 9.525 9.525) (layer Dwgs.User) (width 0.15))
-    (fp_line (start -9.525 -9.525) (end 9.525 -9.525) (layer Dwgs.User) (width 0.15))
-    (fp_line (start -7 -7) (end -7 -5) (layer Dwgs.User) (width 0.15))
-    (fp_line (start -5 -7) (end -7 -7) (layer Dwgs.User) (width 0.15))
-    (fp_line (start -7 7) (end -5 7) (layer Dwgs.User) (width 0.15))
-    (fp_line (start -7 5) (end -7 7) (layer Dwgs.User) (width 0.15))
-    (fp_line (start 7 7) (end 7 5) (layer Dwgs.User) (width 0.15))
-    (fp_line (start 5 7) (end 7 7) (layer Dwgs.User) (width 0.15))
-    (fp_line (start 7 -7) (end 7 -5) (layer Dwgs.User) (width 0.15))
-    (fp_line (start 5 -7) (end 7 -7) (layer Dwgs.User) (width 0.15))
-    (pad "" np_thru_hole circle (at 5.08 0 48.0996) (size 1.75 1.75) (drill 1.75) (layers *.Cu *.Mask))
-    (pad "" np_thru_hole circle (at -5.08 0 48.0996) (size 1.75 1.75) (drill 1.75) (layers *.Cu *.Mask))
-    (pad 1 thru_hole circle (at -2.5 -4) (size 2.25 2.25) (drill 1.47) (layers *.Cu B.Mask)
-      (net 14 "Net-(D13-Pad2)"))
-    (pad "" np_thru_hole circle (at 0 0) (size 3.9878 3.9878) (drill 3.9878) (layers *.Cu *.Mask))
-    (pad 1 thru_hole oval (at -3.81 -2.54 48.0996) (size 4.211556 2.25) (drill 1.47 (offset 0.980778 0)) (layers *.Cu B.Mask)
-      (net 14 "Net-(D13-Pad2)"))
-    (pad 2 thru_hole circle (at 2.54 -5.08) (size 2.25 2.25) (drill 1.47) (layers *.Cu B.Mask)
-      (net 57 COL12))
-    (pad 2 thru_hole oval (at 2.5 -4.5 86.0548) (size 2.831378 2.25) (drill 1.47 (offset 0.290689 0)) (layers *.Cu B.Mask)
-      (net 57 COL12))
-  )
   (module MX_Alps_Hybrid:MX-10U-ReversedStabilizers-NoLED (layer F.Cu)
     (at 148.43125 134.14375)
@@
   (gr_arc (start 17.4625 141.2875) (end 15.08125 141.2875) (angle -90) (layer Edge.Cuts) (width 0.05))
   (gr_arc (start 17.4625 69.85) (end 17.4625 67.46875) (angle -90) (layer Edge.Cuts) (width 0.05))
-  (segment (start 269.24 84.1375) (end 269.71625 84.61375) (width 0.254) (layer B.Cu) (net 0))
-  (segment (start 268.2875 84.1375) (end 269.24 84.1375) (width 0.254) (layer B.Cu) (net 0))
-  (segment (start 268.01126 83.86126) (end 268.2875 84.1375) (width 0.254) (layer B.Cu) (net 0))
+  (segment (start 268.46225 84.61375) (end 269.71625 84.61375) (width 0.254) (layer B.Cu) (net 0))
+  (segment (start 267.70976 83.86126) (end 268.46225 84.61375) (width 0.254) (layer B.Cu) (net 0))
+  (segment (start 38.21749 83.86126) (end 267.70976 83.86126) (width 0.254) (layer B.Cu) (net 0))
   (segment (start 33.3375 88.74125) (end 38.21749 83.86126) (width 0.254) (layer B.Cu) (net 0))
-  (segment (start 38.21749 83.86126) (end 268.01126 83.86126) (width 0.254) (layer B.Cu) (net 0))
   (segment (start 273.716251 83.613751) (end 274.71625 84.61375) (width 0.254) (layer B.Cu) (net 0))
   (segment (start 25.7175 88.74125) (end 25.7175 88.5825) (width 0.254) (layer B.Cu) (net 0))
@@
   (segment (start 251.7925 73.3425) (end 257.96875 73.3425) (width 0.254) (layer B.Cu) (net 13))
   (segment (start 250.94375 72.49375) (end 251.7925 73.3425) (width 0.254) (layer B.Cu) (net 13))
-  (segment (start 269.71625 73.18375) (end 268.44625 74.45375) (width 0.254) (layer B.Cu) (net 14))
-  (segment (start 269.71625 70.11375) (end 269.71625 73.18375) (width 0.254) (layer B.Cu) (net 14))
-  (segment (start 268.44625 74.45375) (end 268.44625 73.9775) (width 0.254) (layer B.Cu) (net 14))
-  (segment (start 267.81125 73.3425) (end 261.14375 73.3425) (width 0.254) (layer B.Cu) (net 14))
-  (segment (start 268.44625 73.9775) (end 267.81125 73.3425) (width 0.254) (layer B.Cu) (net 14))
   (segment (start 35.09875 92.3925) (end 41.275 92.3925) (width 0.254) (layer B.Cu) (net 15))
   (segment (start 34.25 91.54375) (end 35.09875 92.3925) (width 0.254) (layer B.Cu) (net 15))
@@
   (segment (start 38.4175 88.5825) (end 42.06875 84.93125) (width 0.254) (layer B.Cu) (net 56))
   (segment (start 44.45 84.93125) (end 42.06875 84.93125) (width 0.254) (layer B.Cu) (net 56))
+  (segment (start 268.44625 131.45375) (end 268.44625 131.60375) (width 0.254) (layer F.Cu) (net 57))
+  (segment (start 279.13625 120.76375) (end 268.44625 131.45375) (width 0.254) (layer F.Cu) (net 57))
   (segment (start 268.44625 131.60375) (end 268.44625 130.01625) (width 0.254) (layer B.Cu) (net 57))
   (segment (start 268.44625 131.60375) (end 268.44625 130.81) (width 0.254) (layer F.Cu) (net 57))
@@
   (segment (start 36.677499 87.941251) (end 40.30348 84.31527) (width 0.254) (layer B.Cu) (net 57))
   (segment (start 35.8775 88.74125) (end 36.677499 87.941251) (width 0.254) (layer B.Cu) (net 57))
-  (segment (start 274.71625 72.45375) (end 274.75625 72.49375) (width 0.254) (layer B.Cu) (net 57))
-  (segment (start 274.71625 70.11375) (end 274.71625 72.45375) (width 0.254) (layer B.Cu) (net 57))
-  (segment (start 268.44625 131.45375) (end 268.44625 131.60375) (width 0.254) (layer F.Cu) (net 57))
-  (segment (start 277.8125 122.0875) (end 268.44625 131.45375) (width 0.254) (layer F.Cu) (net 57))
-  (segment (start 274.75625 72.49375) (end 274.75625 73.9375) (width 0.254) (layer B.Cu) (net 57))
-  (segment (start 274.75625 73.9375) (end 275.43125 74.6125) (width 0.254) (layer B.Cu) (net 57))
-  (segment (start 275.43125 74.6125) (end 275.43125 79.375) (width 0.254) (layer B.Cu) (net 57))
-  (segment (start 275.43125 79.375) (end 275.43125 80.16875) (width 0.254) (layer B.Cu) (net 57))
-  (segment (start 275.43125 80.16875) (end 277.8125 82.55) (width 0.254) (layer B.Cu) (net 57))
-  (via (at 277.8125 86.51875) (size 0.8) (drill 0.4) (layers F.Cu B.Cu) (net 57))
-  (segment (start 277.8125 82.55) (end 277.8125 86.51875) (width 0.254) (layer B.Cu) (net 57))
-  (segment (start 277.8125 86.51875) (end 277.8125 122.0875) (width 0.254) (layer F.Cu) (net 57))
-  (segment (start 265.754567 86.51875) (end 263.551087 84.31527) (width 0.254) (layer B.Cu) (net 57))
-  (segment (start 277.8125 86.51875) (end 265.754567 86.51875) (width 0.254) (layer B.Cu) (net 57))
-  (segment (start 263.551087 84.31527) (end 40.30348 84.31527) (width 0.254) (layer B.Cu) (net 57))
+  (segment (start 41.89098 84.31527) (end 40.30348 84.31527) (width 0.254) (layer B.Cu) (net 57))
+  (segment (start 264.14098 84.31527) (end 41.89098 84.31527) (width 0.254) (layer B.Cu) (net 57))
   (segment (start 32.7025 112.55375) (end 32.7025 113.665) (width 0.254) (layer F.Cu) (net 58))
   (segment (start 25.55875 74.45375) (end 25.55875 75.565) (width 0.254) (layer F.Cu) (net 58))
@@
   (segment (start 24.917501 93.351249) (end 24.917501 103.181251) (width 0.381) (layer B.Cu) (net 59))
   (segment (start 28.2575 90.01125) (end 24.917501 93.351249) (width 0.381) (layer B.Cu) (net 59))
-  (segment (start 271.4625 83.657098) (end 271.4625 83.86) (width 0.381) (layer B.Cu) (net 59))
+  (segment (start 272.21625 83.30375) (end 272.21625 84.61375) (width 0.381) (layer B.Cu) (net 59))
   (segment (start 33.655 83.34375) (end 268.2875 83.34375) (width 0.381) (layer B.Cu) (net 59))
-  (segment (start 271.4625 83.86) (end 272.21625 84.61375) (width 0.381) (layer B.Cu) (net 59))
   (segment (start 28.2575 88.74125) (end 33.655 83.34375) (width 0.381) (layer B.Cu) (net 59))
   (segment (start 268.2875 83.34375) (end 268.2875 83.339598) (width 0.381) (layer B.Cu) (net 59))
   (segment (start 268.2875 83.339598) (end 268.403849 83.223249) (width 0.381) (layer B.Cu) (net 59))
-  (segment (start 268.403849 83.223249) (end 271.028651 83.223249) (width 0.381) (layer B.Cu) (net 59))
-  (segment (start 271.028651 83.223249) (end 271.4625 83.657098) (width 0.381) (layer B.Cu) (net 59))
+  (segment (start 268.403849 83.223249) (end 272.135749 83.223249) (width 0.381) (layer B.Cu) (net 59))
+  (segment (start 272.135749 83.223249) (end 272.21625 83.30375) (width 0.381) (layer B.Cu) (net 59))
 )
