File: Full-Bar.kicad_pcb (KiCad board)
At the start: 2 copper layers, 83 parts, among them SW1 Rotary_Encoder_Switch, U1 ProMicro

Commit message: Finish layout minus pm
Parts:
- MX1, MX12: footprint MX_Only:MXOnly-1.5U-NoLED -> MX_Alps_Hybrid:MX-1.5U-NoLED
- MX10, MX11, MX14, MX15, MX16, MX17, MX18, MX19, MX2, MX20, MX21, MX22, MX23, MX26, MX27, MX28, MX29, MX3, MX30, MX31, MX32, MX33, MX34, MX36, MX37, MX39, MX4, MX40, MX5, MX6, MX7, MX8, MX9: footprint MX_Only:MXOnly-1U-NoLED -> MX_Alps_Hybrid:MX-1U-NoLED
- MX13: footprint MX_Only:MXOnly-1.75U-NoLED -> MX_Alps_Hybrid:MX-1.75U-NoLED
- MX24, MX25: footprint MX_Only:MXOnly-2.25U-NoLED -> MX_Alps_Hybrid:MX-2.25U-NoLED
- MX35: footprint MX_Only:MXOnly-2.75U-NoLED -> MX_Alps_Hybrid:MX-2.75U-NoLED
- MX38: footprint MX_Only:MXOnly-7U-NoLED -> MX_Alps_Hybrid:MX-10U-NoLED
- U1: moved to B.Cu
- moved D41 262.8 mm to (262.7, 138.1), turned to 90 degrees
- moved D14 258.5 mm to (41.3, 100.0), turned to 90 degrees
- moved D40 238.2 mm to (243.7, 138.1), turned to 90 degrees
- moved D28 233.4 mm to (96.0, 119.1), turned to 90 degrees
- moved D29 228.3 mm to (115.1, 119.1), turned to 90 degrees
- moved D15 223.9 mm to (67.5, 100.0), turned to 90 degrees
- moved D16 215.5 mm to (86.5, 100.0), turned to 90 degrees
- moved D18 211.9 mm to (124.6, 100.0), turned to 90 degrees
- moved D33 211.3 mm to (191.3, 119.1), turned to 90 degrees
- moved D17 208.5 mm to (105.6, 100.0), turned to 90 degrees
- moved D5 203.7 mm to (119.9, 81.0), turned to 90 degrees
- moved D32 187.8 mm to (172.2, 119.1), turned to 90 degrees
- moved D36 183.7 mm to (232.6, 119.1), turned to 90 degrees
- moved D3 175.9 mm to (81.8, 81.0), turned to 90 degrees
- moved D26 174.2 mm to (56.4, 119.1), turned to 90 degrees
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Connections:
- SW1 pad A: ENC1 -> (no net)
- SW1 pad B: ENC0 -> (no net)
- SW1 pad C: GND -> (no net)
- U1 pad 1: Net-(U1-Pad1) -> (no net)
- U1 pad 10: Net-(U1-Pad10) -> (no net)
- U1 pad 11: Net-(U1-Pad11) -> (no net)
- U1 pad 12: Net-(U1-Pad12) -> (no net)
- U1 pad 13: Net-(U1-Pad13) -> (no net)
- U1 pad 14: Net-(U1-Pad14) -> (no net)
- U1 pad 15: Net-(U1-Pad15) -> (no net)
- U1 pad 16: Net-(U1-Pad16) -> (no net)
- U1 pad 17: Net-(U1-Pad17) -> (no net)
- U1 pad 18: Net-(U1-Pad18) -> (no net)
- U1 pad 19: Net-(U1-Pad19) -> (no net)
- U1 pad 2: Net-(U1-Pad2) -> (no net)
- U1 pad 20: Net-(U1-Pad20) -> (no net)
- U1 pad 21: Net-(U1-Pad21) -> (no net)
- U1 pad 22: Net-(U1-Pad22) -> (no net)
- U1 pad 23: Net-(U1-Pad23) -> (no net)
- U1 pad 24: Net-(U1-Pad24) -> (no net)
- U1 pad 3: Net-(U1-Pad3) -> (no net)
- U1 pad 4: Net-(U1-Pad4) -> (no net)
- U1 pad 5: Net-(U1-Pad5) -> (no net)
- U1 pad 6: Net-(U1-Pad6) -> (no net)
- U1 pad 7: Net-(U1-Pad7) -> (no net)
- U1 pad 8: Net-(U1-Pad8) -> (no net)
- U1 pad 9: Net-(U1-Pad9) -> (no net)

Commit message: Pm placed edges defined
Parts:
- MX38: footprint MX_Alps_Hybrid:MX-10U-NoLED -> MX_Alps_Hybrid:MX-10U-ReversedStabilizers-NoLED
- moved U1 68.6 mm to (37.1, 96.4)
- moved D1 2.38 mm to (38.9, 81.0)
Other:
- board outline added: 266.7 x 76.2 mm
Changed lines of the file:
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@@
   (general
     (thickness 1.6)
-    (drawings 0)
+    (drawings 8)
     (tracks 0)
     (zones 0)
@@
     (add_net ROW3)
   )
+  (module MX_Alps_Hybrid:MX-10U-ReversedStabilizers-NoLED (layer F.Cu)
+    (at 148.43125 134.14375)
+    (fp_text reference MX38 (at 0 3.175) (layer Dwgs.User)
+      (effects (font (size 1 1) (thickness 0.15)))
+    )
+    (fp_text value MX-NoLED (at 0 -7.9375) (layer Dwgs.User)
+      (effects (font (size 1 1) (thickness 0.15)))
+    )
+    (fp_line (start -95.25 9.525) (end -95.25 -9.525) (layer Dwgs.User) (width 0.15))
+    (fp_line (start -95.25 9.525) (end 95.25 9.525) (layer Dwgs.User) (width 0.15))
+    (fp_line (start 95.25 -9.525) (end 95.25 9.525) (layer Dwgs.User) (width 0.15))
+    (fp_line (start -95.25 -9.525) (end 95.25 -9.525) (layer Dwgs.User) (width 0.15))
+    (fp_line (start -7 -7) (end -7 -5) (layer Dwgs.User) (width 0.15))
+    (fp_line (start -5 -7) (end -7 -7) (layer Dwgs.User) (width 0.15))
+    (fp_line (start -7 7) (end -5 7) (layer Dwgs.User) (width 0.15))
+    (fp_line (start -7 5) (end -7 7) (layer Dwgs.User) (width 0.15))
+    (fp_line (start 7 7) (end 7 5) (layer Dwgs.User) (width 0.15))
+    (fp_line (start 5 7) (end 7 7) (layer Dwgs.User) (width 0.15))
+    (fp_line (start 7 -7) (end 7 -5) (layer Dwgs.User) (width 0.15))
+    (fp_line (start 5 -7) (end 7 -7) (layer Dwgs.User) (width 0.15))
+    (pad "" np_thru_hole circle (at 66.675 -8.255) (size 3.9878 3.9878) (drill 3.9878) (layers *.Cu *.Mask))
+    (pad "" np_thru_hole circle (at -66.675 -8.255) (size 3.9878 3.9878) (drill 3.9878) (layers *.Cu *.Mask))
+    (pad "" np_thru_hole circle (at 66.675 6.985) (size 3.048 3.048) (drill 3.048) (layers *.Cu *.Mask))
+    (pad "" np_thru_hole circle (at -66.675 6.985) (size 3.048 3.048) (drill 3.048) (layers *.Cu *.Mask))
+    (pad "" np_thru_hole circle (at 5.08 0 48.0996) (size 1.75 1.75) (drill 1.75) (layers *.Cu *.Mask))
+    (pad "" np_thru_hole circle (at -5.08 0 48.0996) (size 1.75 1.75) (drill 1.75) (layers *.Cu *.Mask))
+    (pad 1 thru_hole circle (at -2.5 -4) (size 2.25 2.25) (drill 1.47) (layers *.Cu B.Mask)
+      (net 51 COL6))
+    (pad "" np_thru_hole circle (at 0 0) (size 3.9878 3.9878) (drill 3.9878) (layers *.Cu *.Mask))
+    (pad 1 thru_hole oval (at -3.81 -2.54 48.0996) (size 4.211556 2.25) (drill 1.47 (offset 0.980778 0)) (layers *.Cu B.Mask)
+      (net 51 COL6))
+    (pad 2 thru_hole circle (at 2.54 -5.08) (size 2.25 2.25) (drill 1.47) (layers *.Cu B.Mask)
+      (net 43 "Net-(D39-Pad2)"))
+    (pad 2 thru_hole oval (at 2.5 -4.5 86.0548) (size 2.831378 2.25) (drill 1.47 (offset 0.290689 0)) (layers *.Cu B.Mask)
+      (net 43 "Net-(D39-Pad2)"))
+  )
   (module Rotary_Encoder:RotaryEncoder_Alps_EC11E-Switch_Vertical_H20mm (layer F.Cu)
     (at 272.25625 76.99375)
@@
       (net 44 "Net-(D40-Pad2)"))
   )
-  (module MX_Alps_Hybrid:MX-10U-NoLED (layer F.Cu)
-    (at 148.43125 134.14375)
-    (fp_text reference MX38 (at 0 3.175) (layer Dwgs.User)
-      (effects (font (size 1 1) (thickness 0.15)))
-    )
-    (fp_text value MX-NoLED (at 0 -7.9375) (layer Dwgs.User)
-      (effects (font (size 1 1) (thickness 0.15)))
-    )
-    (fp_line (start -95.25 9.525) (end -95.25 -9.525) (layer Dwgs.User) (width 0.15))
-    (fp_line (start -95.25 9.525) (end 95.25 9.525) (layer Dwgs.User) (width 0.15))
-    (fp_line (start 95.25 -9.525) (end 95.25 9.525) (layer Dwgs.User) (width 0.15))
-    (fp_line (start -95.25 -9.525) (end 95.25 -9.525) (layer Dwgs.User) (width 0.15))
-    (fp_line (start -7 -7) (end -7 -5) (layer Dwgs.User) (width 0.15))
-    (fp_line (start -5 -7) (end -7 -7) (layer Dwgs.User) (width 0.15))
-    (fp_line (start -7 7) (end -5 7) (layer Dwgs.User) (width 0.15))
-    (fp_line (start -7 5) (end -7 7) (layer Dwgs.User) (width 0.15))
-    (fp_line (start 7 7) (end 7 5) (layer Dwgs.User) (width 0.15))
-    (fp_line (start 5 7) (end 7 7) (layer Dwgs.User) (width 0.15))
-    (fp_line (start 7 -7) (end 7 -5) (layer Dwgs.User) (width 0.15))
-    (fp_line (start 5 -7) (end 7 -7) (layer Dwgs.User) (width 0.15))
-    (pad "" np_thru_hole circle (at 66.675 8.255) (size 3.9878 3.9878) (drill 3.9878) (layers *.Cu *.Mask))
-    (pad "" np_thru_hole circle (at -66.675 8.255) (size 3.9878 3.9878) (drill 3.9878) (layers *.Cu *.Mask))
-    (pad "" np_thru_hole circle (at 66.675 -6.985) (size 3.048 3.048) (drill 3.048) (layers *.Cu *.Mask))
-    (pad "" np_thru_hole circle (at -66.675 -6.985) (size 3.048 3.048) (drill 3.048) (layers *.Cu *.Mask))
-    (pad "" np_thru_hole circle (at 5.08 0 48.0996) (size 1.75 1.75) (drill 1.75) (layers *.Cu *.Mask))
-    (pad "" np_thru_hole circle (at -5.08 0 48.0996) (size 1.75 1.75) (drill 1.75) (layers *.Cu *.Mask))
-    (pad 1 thru_hole circle (at -2.5 -4) (size 2.25 2.25) (drill 1.47) (layers *.Cu B.Mask)
-      (net 51 COL6))
-    (pad "" np_thru_hole circle (at 0 0) (size 3.9878 3.9878) (drill 3.9878) (layers *.Cu *.Mask))
-    (pad 1 thru_hole oval (at -3.81 -2.54 48.0996) (size 4.211556 2.25) (drill 1.47 (offset 0.980778 0)) (layers *.Cu B.Mask)
-      (net 51 COL6))
-    (pad 2 thru_hole circle (at 2.54 -5.08) (size 2.25 2.25) (drill 1.47) (layers *.Cu B.Mask)
-      (net 43 "Net-(D39-Pad2)"))
-    (pad 2 thru_hole oval (at 2.5 -4.5 86.0548) (size 2.831378 2.25) (drill 1.47 (offset 0.290689 0)) (layers *.Cu B.Mask)
-      (net 43 "Net-(D39-Pad2)"))
-  )
   (module MX_Alps_Hybrid:MX-1U-NoLED (layer F.Cu)
     (at 43.65625 134.14375)
@@
   )
   (module promicro:ProMicro (layer B.Cu)
-    (at 74.6125 38.89375)
+    (at 37.1475 96.36125)
     (descr "Pro Micro footprint")
     (tags "promicro ProMicro")
@@
   )
   (module Diode_THT:D_A-405_P7.62mm_Horizontal (layer F.Cu)
-    (at 41.275 80.9625 90)
+    (at 38.89375 80.9625 90)
     (descr "Diode, A-405 series, Axial, Horizontal, pin pitch=7.62mm, , length*diameter=5.2*2.7mm^2, , http://www.diodes.com/_files/packages/A-405.pdf")
     (tags "Diode A-405 series Axial Horizontal pin pitch 7.62mm  length 5.2mm diameter 2.7mm")
@@
     )
   )
+  (gr_line (start 17.4625 67.46875) (end 279.4 67.46875) (layer Edge.Cuts) (width 0.05))
+  (gr_line (start 15.08125 141.2875) (end 15.08125 69.85) (layer Edge.Cuts) (width 0.05))
+  (gr_line (start 279.4 143.66875) (end 17.4625 143.66875) (layer Edge.Cuts) (width 0.05))
+  (gr_line (start 281.78125 69.85) (end 281.78125 141.2875) (layer Edge.Cuts) (width 0.05))
+  (gr_arc (start 279.4 69.85) (end 281.78125 69.85) (angle -90) (layer Edge.Cuts) (width 0.05))
+  (gr_arc (start 279.4 141.2875) (end 279.4 143.66875) (angle -90) (layer Edge.Cuts) (width 0.05))
+  (gr_arc (start 17.4625 141.2875) (end 15.08125 141.2875) (angle -90) (layer Edge.Cuts) (width 0.05))
+  (gr_arc (start 17.4625 69.85) (end 17.4625 67.46875) (angle -90) (layer Edge.Cuts) (width 0.05))
 )

Commit message: Starting traces
Connections:
- SW1 pad C: (no net) -> GND
- U1 pad 23: (no net) -> GND
- U1 pad 3: (no net) -> GND
- U1 pad 4: (no net) -> GND
Routing:
- net COL1: track 0.00 -> 86.6 mm
- net COL6: track 0.00 -> 63.2 mm
- net COL12: track 0.00 -> 61.2 mm
- net COL13: track 0.00 -> 56.6 mm
- net COL2: track 0.00 -> 45.1 mm
- net COL4: track 0.00 -> 44.4 mm
- net COL8: track 0.00 -> 43.1 mm
- net COL5: track 0.00 -> 43.1 mm
- net COL3: track 0.00 -> 43.1 mm
- net COL9: track 0.00 -> 43.1 mm
- net COL10: track 0.00 -> 43.1 mm
- net COL7: track 0.00 -> 43.1 mm
- net COL11: track 0.00 -> 20.1 mm
Other:
- net class Default: trace_width 0.25 -> 0.254
- net class Power added: clearance 0.2, trace_width 0.381, via_dia 0.8, via_drill 0.4

Commit message: Traces mostly finished minus one column
Routing:
- net (no net): track 0.00 -> 488.2 mm
- net ROW3: track 0.00 -> 277.3 mm
- net GND: track 0.00 -> 265.0 mm
- net COL13: track 56.6 -> 305.3 mm
- net COL12: track 61.2 -> 305.4 mm
- net ROW0: track 0.00 -> 237.7 mm
- net ROW1: track 0.00 -> 205.0 mm
- net ROW2: track 0.00 -> 200.9 mm
- net COL11: track 20.1 -> 209.0 mm
- net COL10: track 43.1 -> 210.2 mm
- net COL9: track 43.1 -> 188.4 mm
- net COL8: track 43.1 -> 166.6 mm
- net COL7: track 43.1 -> 145.1 mm
- net COL6: track 63.2 -> 160.0 mm, vias 0 -> 1
- net COL5: track 43.1 -> 119.1 mm, vias 0 -> 1
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
Commit message: traces ran
Parts:
- added MX41: MX-NoLED, MX_Alps_Hybrid:MX-1U-NoLED, F.Cu at (272.3, 77.0)
- added MX42: MX-NoLED, MX_Alps_Hybrid:MX-7U-ReversedStabilizers-NoLED, F.Cu at (148.4, 134.1)
- turned SW1 to 90 degrees
Connections:
- MX1 pad 1: COL1 -> COL0
- MX10 pad 1: COL10 -> COL9
- MX11 pad 1: COL11 -> COL10
- MX12 pad 1: COL12 -> COL11
- MX13 pad 1: COL1 -> COL0
- MX14 pad 1: COL2 -> COL1
- MX15 pad 1: COL3 -> COL2
- MX16 pad 1: COL4 -> COL3
- MX17 pad 1: COL5 -> COL4
- MX18 pad 1: COL6 -> COL5
- MX19 pad 1: COL7 -> COL6
- MX2 pad 1: COL2 -> COL1
- MX20 pad 1: COL8 -> COL7
- MX21 pad 1: COL9 -> COL8
- MX22 pad 1: COL10 -> COL9
- MX23 pad 1: COL11 -> COL10
- MX24 pad 1: COL12 -> COL11
- MX25 pad 1: COL1 -> COL0
- MX26 pad 1: COL2 -> COL1
- MX27 pad 1: COL3 -> COL2
- MX28 pad 1: COL4 -> COL3
- MX29 pad 1: COL5 -> COL4
- MX3 pad 1: COL3 -> COL2
- MX30 pad 1: COL6 -> COL5
- MX31 pad 1: COL7 -> COL6
- MX32 pad 1: COL8 -> COL7
- MX33 pad 1: COL9 -> COL8
- MX34 pad 1: COL10 -> COL9
- MX35 pad 1: COL12 -> COL11
- MX38 pad 1: COL6 -> COL5
- MX39 pad 1: COL12 -> COL11
- MX4 pad 1: COL4 -> COL3
- MX40 pad 1: COL13 -> COL12
- MX5 pad 1: COL5 -> COL4
- MX6 pad 1: COL6 -> COL5
- MX7 pad 1: COL7 -> COL6
- MX8 pad 1: COL8 -> COL7
- MX9 pad 1: COL9 -> COL8
- SW1 pad S1: COL13 -> COL12
- U1 pad 1: (no net) -> ROW0
- U1 pad 10: (no net) -> COL8
- U1 pad 11: (no net) -> COL7
- U1 pad 12: (no net) -> COL6
- U1 pad 13: (no net) -> COL3
- U1 pad 14: (no net) -> COL4
- U1 pad 15: (no net) -> COL5
- U1 pad 16: (no net) -> COL2
- U1 pad 17: (no net) -> COL1
- U1 pad 18: (no net) -> ROW1
- U1 pad 19: (no net) -> ROW2
- U1 pad 20: (no net) -> ROW3
- U1 pad 24: (no net) -> COL0
- U1 pad 6: (no net) -> COL12
- U1 pad 7: (no net) -> COL11
- U1 pad 8: (no net) -> COL10
- U1 pad 9: (no net) -> COL9
Routing:
- net COL13: track 305.3 -> 0.00 mm
- net COL11: track 209.0 -> 306.6 mm
- net COL0: track 26.6 -> 86.4 mm
- net COL5: track 119.1 -> 161.6 mm
- net COL1: track 70.0 -> 108.1 mm, vias 0 -> 1
- net COL9: track 188.4 -> 211.7 mm
- net COL8: track 166.6 -> 189.8 mm
- net COL7: track 145.1 -> 167.8 mm
- net COL4: track 99.4 -> 120.8 mm
- net COL2: track 69.6 -> 87.8 mm
- net COL3: track 85.8 -> 101.1 mm, vias 0 -> 1
- net COL6: track 160.0 -> 147.0 mm, vias 1 -> 0
- net COL12: track 305.4 -> 314.0 mm, vias 0 -> 1
- net Net-(D13-Pad2): track 21.1 -> 12.9 mm
- net ROW0: track 237.7 -> 241.2 mm
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- added copper zone on B.Cu, net GND
Other:
- board text added: "10upset <3"
