File: Full-Bar.sch (KiCad schematic (older format))
At the start: 83 parts, among them SW1 Rotary_Encoder_Switch, U1 ProMicro

Commit message: Footprint assignments
Parts:
- MX1, MX12: footprint (none) -> MX_Only:MXOnly-1.5U-NoLED
- MX10, MX11, MX14, MX15, MX16, MX17, MX18, MX19, MX2, MX20, MX21, MX22, MX23, MX26, MX27, MX28, MX29, MX3, MX30, MX31, MX32, MX33, MX34, MX36, MX37, MX39, MX4, MX40, MX5, MX6, MX7, MX8, MX9: footprint (none) -> MX_Only:MXOnly-1U-NoLED
- MX13: footprint (none) -> MX_Only:MXOnly-1.75U-NoLED
- MX24, MX25: footprint (none) -> MX_Only:MXOnly-2.25U-NoLED
- MX35: footprint (none) -> MX_Only:MXOnly-2.75U-NoLED
- MX38: footprint (none) -> MX_Only:MXOnly-7U-NoLED
- SW1: footprint (none) -> Rotary_Encoder:RotaryEncoder_Alps_EC11E-Switch_Vertical_H20mm
- U1: footprint (none) -> promicro:ProMicro
Changed lines of the file:
@@
 F 0 "U1" H 3250 8287 60  0000 C CNN
 F 1 "ProMicro" H 3250 8181 60  0000 C CNN
-F 2 "" H 3350 6200 60  0001 C CNN
+F 2 "promicro:ProMicro" H 3350 6200 60  0001 C CNN
 F 3 "" H 3350 6200 60  0000 C CNN
 	1    3250 7250
@@
 F 0 "MX1" H 1733 1323 60  0000 C CNN
 F 1 "MX-NoLED" H 1733 1249 20  0000 C CNN
-F 2 "" H 1075 1075 60  0001 C CNN
+F 2 "MX_Only:MXOnly-1.5U-NoLED" H 1075 1075 60  0001 C CNN
 F 3 "" H 1075 1075 60  0001 C CNN
 	1    1700 1100
@@
 F 0 "MX2" H 2233 1323 60  0000 C CNN
 F 1 "MX-NoLED" H 2233 1249 20  0000 C CNN
-F 2 "" H 1575 1075 60  0001 C CNN
+F 2 "MX_Only:MXOnly-1U-NoLED" H 1575 1075 60  0001 C CNN
 F 3 "" H 1575 1075 60  0001 C CNN
 	1    2200 1100
@@
 F 0 "MX3" H 2733 1323 60  0000 C CNN
 F 1 "MX-NoLED" H 2733 1249 20  0000 C CNN
-F 2 "" H 2075 1075 60  0001 C CNN
+F 2 "MX_Only:MXOnly-1U-NoLED" H 2075 1075 60  0001 C CNN
 F 3 "" H 2075 1075 60  0001 C CNN
 	1    2700 1100
@@
 F 0 "MX4" H 3233 1323 60  0000 C CNN
 F 1 "MX-NoLED" H 3233 1249 20  0000 C CNN
-F 2 "" H 2575 1075 60  0001 C CNN
+F 2 "MX_Only:MXOnly-1U-NoLED" H 2575 1075 60  0001 C CNN
 F 3 "" H 2575 1075 60  0001 C CNN
 	1    3200 1100
@@
 F 0 "MX5" H 3733 1323 60  0000 C CNN
 F 1 "MX-NoLED" H 3733 1249 20  0000 C CNN
-F 2 "" H 3075 1075 60  0001 C CNN
+F 2 "MX_Only:MXOnly-1U-NoLED" H 3075 1075 60  0001 C CNN
 F 3 "" H 3075 1075 60  0001 C CNN
 	1    3700 1100
@@
 F 0 "MX6" H 4233 1323 60  0000 C CNN
 F 1 "MX-NoLED" H 4233 1249 20  0000 C CNN
-F 2 "" H 3575 1075 60  0001 C CNN
+F 2 "MX_Only:MXOnly-1U-NoLED" H 3575 1075 60  0001 C CNN
 F 3 "" H 3575 1075 60  0001 C CNN
 	1    4200 1100
@@
 F 0 "MX7" H 4733 1323 60  0000 C CNN
 F 1 "MX-NoLED" H 4733 1249 20  0000 C CNN
-F 2 "" H 4075 1075 60  0001 C CNN
+F 2 "MX_Only:MXOnly-1U-NoLED" H 4075 1075 60  0001 C CNN
 F 3 "" H 4075 1075 60  0001 C CNN
 	1    4700 1100
@@
 F 0 "MX8" H 5233 1323 60  0000 C CNN
 F 1 "MX-NoLED" H 5233 1249 20  0000 C CNN
-F 2 "" H 4575 1075 60  0001 C CNN
+F 2 "MX_Only:MXOnly-1U-NoLED" H 4575 1075 60  0001 C CNN
 F 3 "" H 4575 1075 60  0001 C CNN
 	1    5200 1100
@@
 F 0 "MX9" H 5733 1323 60  0000 C CNN
 F 1 "MX-NoLED" H 5733 1249 20  0000 C CNN
-F 2 "" H 5075 1075 60  0001 C CNN
+F 2 "MX_Only:MXOnly-1U-NoLED" H 5075 1075 60  0001 C CNN
 F 3 "" H 5075 1075 60  0001 C CNN
 	1    5700 1100
@@
 F 0 "MX10" H 6233 1323 60  0000 C CNN
 F 1 "MX-NoLED" H 6233 1249 20  0000 C CNN
-F 2 "" H 5575 1075 60  0001 C CNN
+F 2 "MX_Only:MXOnly-1U-NoLED" H 5575 1075 60  0001 C CNN
 F 3 "" H 5575 1075 60  0001 C CNN
 	1    6200 1100
@@
 F 0 "MX11" H 6733 1323 60  0000 C CNN
 F 1 "MX-NoLED" H 6733 1249 20  0000 C CNN
-F 2 "" H 6075 1075 60  0001 C CNN
+F 2 "MX_Only:MXOnly-1U-NoLED" H 6075 1075 60  0001 C CNN
 F 3 "" H 6075 1075 60  0001 C CNN
 	1    6700 1100
@@
 F 0 "MX12" H 7233 1323 60  0000 C CNN
 F 1 "MX-NoLED" H 7233 1249 20  0000 C CNN
-F 2 "" H 6575 1075 60  0001 C CNN
+F 2 "MX_Only:MXOnly-1.5U-NoLED" H 6575 1075 60  0001 C CNN
 F 3 "" H 6575 1075 60  0001 C CNN
 	1    7200 1100
@@
 F 0 "SW1" H 7900 1517 50  0000 C CNN
 F 1 "Rotary_Encoder_Switch" H 7900 1426 50  0000 C CNN
-F 2 "" H 7750 1310 50  0001 C CNN
+F 2 "Rotary_Encoder:RotaryEncoder_Alps_EC11E-Switch_Vertical_H20mm" H 7750 1310 50  0001 C CNN
 F 3 "~" H 7900 1410 50  0001 C CNN
 	1    7900 1150
@@
 F 0 "MX13" H 1733 1973 60  0000 C CNN
 F 1 "MX-NoLED" H 1733 1899 20  0000 C CNN
-F 2 "" H 1075 1725 60  0001 C CNN
+F 2 "MX_Only:MXOnly-1.75U-NoLED" H 1075 1725 60  0001 C CNN
 F 3 "" H 1075 1725 60  0001 C CNN
 	1    1700 1750
@@
 F 0 "MX14" H 2233 1973 60  0000 C CNN
 F 1 "MX-NoLED" H 2233 1899 20  0000 C CNN
-F 2 "" H 1575 1725 60  0001 C CNN
+F 2 "MX_Only:MXOnly-1U-NoLED" H 1575 1725 60  0001 C CNN
 F 3 "" H 1575 1725 60  0001 C CNN
 	1    2200 1750
@@
 F 0 "MX15" H 2733 1973 60  0000 C CNN
 F 1 "MX-NoLED" H 2733 1899 20  0000 C CNN
-F 2 "" H 2075 1725 60  0001 C CNN
+F 2 "MX_Only:MXOnly-1U-NoLED" H 2075 1725 60  0001 C CNN
 F 3 "" H 2075 1725 60  0001 C CNN
 	1    2700 1750
@@
 F 0 "MX16" H 3233 1973 60  0000 C CNN
 F 1 "MX-NoLED" H 3233 1899 20  0000 C CNN
-F 2 "" H 2575 1725 60  0001 C CNN
+F 2 "MX_Only:MXOnly-1U-NoLED" H 2575 1725 60  0001 C CNN
 F 3 "" H 2575 1725 60  0001 C CNN
 	1    3200 1750
@@
 F 0 "MX17" H 3733 1973 60  0000 C CNN
 F 1 "MX-NoLED" H 3733 1899 20  0000 C CNN
-F 2 "" H 3075 1725 60  0001 C CNN
+F 2 "MX_Only:MXOnly-1U-NoLED" H 3075 1725 60  0001 C CNN
 F 3 "" H 3075 1725 60  0001 C CNN
 	1    3700 1750
@@
 F 0 "MX18" H 4233 1973 60  0000 C CNN
 F 1 "MX-NoLED" H 4233 1899 20  0000 C CNN
-F 2 "" H 3575 1725 60  0001 C CNN
+F 2 "MX_Only:MXOnly-1U-NoLED" H 3575 1725 60  0001 C CNN
 F 3 "" H 3575 1725 60  0001 C CNN
 	1    4200 1750
@@
 F 0 "MX19" H 4733 1973 60  0000 C CNN
 F 1 "MX-NoLED" H 4733 1899 20  0000 C CNN
-F 2 "" H 4075 1725 60  0001 C CNN
+F 2 "MX_Only:MXOnly-1U-NoLED" H 4075 1725 60  0001 C CNN
 F 3 "" H 4075 1725 60  0001 C CNN
 	1    4700 1750
@@
 F 0 "MX20" H 5233 1973 60  0000 C CNN
 F 1 "MX-NoLED" H 5233 1899 20  0000 C CNN
-F 2 "" H 4575 1725 60  0001 C CNN
+F 2 "MX_Only:MXOnly-1U-NoLED" H 4575 1725 60  0001 C CNN
 F 3 "" H 4575 1725 60  0001 C CNN
 	1    5200 1750
@@
 F 0 "MX21" H 5733 1973 60  0000 C CNN
 F 1 "MX-NoLED" H 5733 1899 20  0000 C CNN
-F 2 "" H 5075 1725 60  0001 C CNN
+F 2 "MX_Only:MXOnly-1U-NoLED" H 5075 1725 60  0001 C CNN
 F 3 "" H 5075 1725 60  0001 C CNN
 	1    5700 1750
@@
 F 0 "MX22" H 6233 1973 60  0000 C CNN
 F 1 "MX-NoLED" H 6233 1899 20  0000 C CNN
-F 2 "" H 5575 1725 60  0001 C CNN
+F 2 "MX_Only:MXOnly-1U-NoLED" H 5575 1725 60  0001 C CNN
 F 3 "" H 5575 1725 60  0001 C CNN
 	1    6200 1750
@@
 F 0 "MX23" H 6733 1973 60  0000 C CNN
 F 1 "MX-NoLED" H 6733 1899 20  0000 C CNN
-F 2 "" H 6075 1725 60  0001 C CNN
+F 2 "MX_Only:MXOnly-1U-NoLED" H 6075 1725 60  0001 C CNN
 F 3 "" H 6075 1725 60  0001 C CNN
 	1    6700 1750
@@
 F 0 "MX24" H 7233 1973 60  0000 C CNN
 F 1 "MX-NoLED" H 7233 1899 20  0000 C CNN
-F 2 "" H 6575 1725 60  0001 C CNN
+F 2 "MX_Only:MXOnly-2.25U-NoLED" H 6575 1725 60  0001 C CNN
 F 3 "" H 6575 1725 60  0001 C CNN
 	1    7200 1750
@@
 F 0 "MX25" H 1733 2623 60  0000 C CNN
 F 1 "MX-NoLED" H 1733 2549 20  0000 C CNN
-F 2 "" H 1075 2375 60  0001 C CNN
+F 2 "MX_Only:MXOnly-2.25U-NoLED" H 1075 2375 60  0001 C CNN
 F 3 "" H 1075 2375 60  0001 C CNN
 	1    1700 2400
@@
 F 0 "MX26" H 2233 2623 60  0000 C CNN
 F 1 "MX-NoLED" H 2233 2549 20  0000 C CNN
-F 2 "" H 1575 2375 60  0001 C CNN
+F 2 "MX_Only:MXOnly-1U-NoLED" H 1575 2375 60  0001 C CNN
 F 3 "" H 1575 2375 60  0001 C CNN
 	1    2200 2400
@@
 F 0 "MX27" H 2733 2623 60  0000 C CNN
 F 1 "MX-NoLED" H 2733 2549 20  0000 C CNN
-F 2 "" H 2075 2375 60  0001 C CNN
+F 2 "MX_Only:MXOnly-1U-NoLED" H 2075 2375 60  0001 C CNN
 F 3 "" H 2075 2375 60  0001 C CNN
 	1    2700 2400
@@
 F 0 "MX28" H 3233 2623 60  0000 C CNN
 F 1 "MX-NoLED" H 3233 2549 20  0000 C CNN
-F 2 "" H 2575 2375 60  0001 C CNN
+F 2 "MX_Only:MXOnly-1U-NoLED" H 2575 2375 60  0001 C CNN
 F 3 "" H 2575 2375 60  0001 C CNN
 	1    3200 2400
@@
 F 0 "MX29" H 3733 2623 60  0000 C CNN
 F 1 "MX-NoLED" H 3733 2549 20  0000 C CNN
-F 2 "" H 3075 2375 60  0001 C CNN
+F 2 "MX_Only:MXOnly-1U-NoLED" H 3075 2375 60  0001 C CNN
 F 3 "" H 3075 2375 60  0001 C CNN
 	1    3700 2400
@@
 F 0 "MX30" H 4233 2623 60  0000 C CNN
 F 1 "MX-NoLED" H 4233 2549 20  0000 C CNN
-F 2 "" H 3575 2375 60  0001 C CNN
+F 2 "MX_Only:MXOnly-1U-NoLED" H 3575 2375 60  0001 C CNN
 F 3 "" H 3575 2375 60  0001 C CNN
 	1    4200 2400
@@
 F 0 "MX31" H 4733 2623 60  0000 C CNN
 F 1 "MX-NoLED" H 4733 2549 20  0000 C CNN
-F 2 "" H 4075 2375 60  0001 C CNN
+F 2 "MX_Only:MXOnly-1U-NoLED" H 4075 2375 60  0001 C CNN
 F 3 "" H 4075 2375 60  0001 C CNN
 	1    4700 2400
@@
 F 0 "MX32" H 5233 2623 60  0000 C CNN
 F 1 "MX-NoLED" H 5233 2549 20  0000 C CNN
-F 2 "" H 4575 2375 60  0001 C CNN
+F 2 "MX_Only:MXOnly-1U-NoLED" H 4575 2375 60  0001 C CNN
 F 3 "" H 4575 2375 60  0001 C CNN
 	1    5200 2400
@@
 F 0 "MX33" H 5733 2623 60  0000 C CNN
 F 1 "MX-NoLED" H 5733 2549 20  0000 C CNN
-F 2 "" H 5075 2375 60  0001 C CNN
+F 2 "MX_Only:MXOnly-1U-NoLED" H 5075 2375 60  0001 C CNN
 F 3 "" H 5075 2375 60  0001 C CNN
 	1    5700 2400
@@
 F 0 "MX34" H 6233 2623 60  0000 C CNN
 F 1 "MX-NoLED" H 6233 2549 20  0000 C CNN
-F 2 "" H 5575 2375 60  0001 C CNN
+F 2 "MX_Only:MXOnly-1U-NoLED" H 5575 2375 60  0001 C CNN
 F 3 "" H 5575 2375 60  0001 C CNN
 	1    6200 2400
@@
 F 0 "MX35" H 7233 2623 60  0000 C CNN
 F 1 "MX-NoLED" H 7233 2549 20  0000 C CNN
-F 2 "" H 6575 2375 60  0001 C CNN
+F 2 "MX_Only:MXOnly-2.75U-NoLED" H 6575 2375 60  0001 C CNN
 F 3 "" H 6575 2375 60  0001 C CNN
 	1    7200 2400
@@
 F 0 "MX36" H 1233 3273 60  0000 C CNN
 F 1 "MX-NoLED" H 1233 3199 20  0000 C CNN
-F 2 "" H 575 3025 60  0001 C CNN
+F 2 "MX_Only:MXOnly-1U-NoLED" H 575 3025 60  0001 C CNN
 F 3 "" H 575 3025 60  0001 C CNN
 	1    1200 3050
@@
 F 0 "MX37" H 1733 3273 60  0000 C CNN
 F 1 "MX-NoLED" H 1733 3199 20  0000 C CNN
-F 2 "" H 1075 3025 60  0001 C CNN
+F 2 "MX_Only:MXOnly-1U-NoLED" H 1075 3025 60  0001 C CNN
 F 3 "" H 1075 3025 60  0001 C CNN
 	1    1700 3050
@@
 F 0 "MX38" H 4233 3273 60  0000 C CNN
 F 1 "MX-NoLED" H 4233 3199 20  0000 C CNN
-F 2 "" H 3575 3025 60  0001 C CNN
+F 2 "MX_Only:MXOnly-7U-NoLED" H 3575 3025 60  0001 C CNN
 F 3 "" H 3575 3025 60  0001 C CNN
 	1    4200 3050
@@
 F 0 "MX39" H 7233 3273 60  0000 C CNN
 F 1 "MX-NoLED" H 7233 3199 20  0000 C CNN
-F 2 "" H 6575 3025 60  0001 C CNN
+F 2 "MX_Only:MXOnly-1U-NoLED" H 6575 3025 60  0001 C CNN
 F 3 "" H 6575 3025 60  0001 C CNN
 	1    7200 3050
@@
 F 0 "MX40" H 8083 3273 60  0000 C CNN
 F 1 "MX-NoLED" H 8083 3199 20  0000 C CNN
-F 2 "" H 7425 3025 60  0001 C CNN
+F 2 "MX_Only:MXOnly-1U-NoLED" H 7425 3025 60  0001 C CNN
 F 3 "" H 7425 3025 60  0001 C CNN
 	1    8050 3050

Commit message: Pcb start
Parts:
- D1, D10, D11, D12, D13, D14, D15, D16, D17, D18, D19, D2, D20, D21, D22, D23, D24, D25, D26, D27, D28, D29, D3, D30, D31, D32, D33, D34, D35, D36, D37, D38, D39, D4, D40, D41, D5, D6, D7, D8, D9: footprint Diode_THT:D_5KP_P10.16mm_Horizontal -> Diode_THT:D_A-405_P7.62mm_Horizontal

Commit message: Finish layout minus pm
Parts:
- MX1, MX12: footprint MX_Only:MXOnly-1.5U-NoLED -> MX_Alps_Hybrid:MX-1.5U-NoLED
- MX10, MX11, MX14, MX15, MX16, MX17, MX18, MX19, MX2, MX20, MX21, MX22, MX23, MX26, MX27, MX28, MX29, MX3, MX30, MX31, MX32, MX33, MX34, MX36, MX37, MX39, MX4, MX40, MX5, MX6, MX7, MX8, MX9: footprint MX_Only:MXOnly-1U-NoLED -> MX_Alps_Hybrid:MX-1U-NoLED
- MX13: footprint MX_Only:MXOnly-1.75U-NoLED -> MX_Alps_Hybrid:MX-1.75U-NoLED
- MX24, MX25: footprint MX_Only:MXOnly-2.25U-NoLED -> MX_Alps_Hybrid:MX-2.25U-NoLED
- MX35: footprint MX_Only:MXOnly-2.75U-NoLED -> MX_Alps_Hybrid:MX-2.75U-NoLED
- MX38: footprint MX_Only:MXOnly-7U-NoLED -> MX_Alps_Hybrid:MX-10U-NoLED

Commit message: Pm placed edges defined
Parts:
- MX38: footprint MX_Alps_Hybrid:MX-10U-NoLED -> MX_Alps_Hybrid:MX-10U-ReversedStabilizers-NoLED
Changed lines of the file:
@@
 F 0 "MX38" H 4233 3273 60  0000 C CNN
 F 1 "MX-NoLED" H 4233 3199 20  0000 C CNN
-F 2 "MX_Alps_Hybrid:MX-10U-NoLED" H 3575 3025 60  0001 C CNN
+F 2 "MX_Alps_Hybrid:MX-10U-ReversedStabilizers-NoLED" H 3575 3025 60  0001 C CNN
 F 3 "" H 3575 3025 60  0001 C CNN
 	1    4200 3050

Commit message: Starting traces
Connections:
- net GND: now also U1.23 (GND), U1.3 (GND), U1.4 (GND)
Changed lines of the file:
@@
 	7500 1150 7500 1850
-Wire Wire Line
-	7500 1850 7850 1850
 Wire Wire Line
 	7600 1250 7600 1750
 Wire Wire Line
 	7600 1750 7850 1750
-Text GLabel 7850 1850 2    50   Input ~ 0
-GND
 Text GLabel 7850 1750 2    50   Input ~ 0
 ENC0
@@
 	0    -1   -1   0
 $EndComp
+$Comp
+L power:GND #PWR0101
+U 1 1 619FAABC
+P 7850 1850
+F 0 "#PWR0101" H 7850 1600 50  0001 C CNN
+F 1 "GND" V 7855 1722 50  0000 R CNN
+F 2 "" H 7850 1850 50  0001 C CNN
+F 3 "" H 7850 1850 50  0001 C CNN
+	1    7850 1850
+	0    -1   -1   0
+$EndComp
+Wire Wire Line
+	7500 1850 7850 1850
+$Comp
+L power:GND #PWR0102
+U 1 1 61A0676F
+P 3950 6600
+F 0 "#PWR0102" H 3950 6350 50  0001 C CNN
+F 1 "GND" V 3955 6472 50  0000 R CNN
+F 2 "" H 3950 6600 50  0001 C CNN
+F 3 "" H 3950 6600 50  0001 C CNN
+	1    3950 6600
+	0    -1   -1   0
+$EndComp
+$Comp
+L power:GND #PWR0103
+U 1 1 61A0D499
+P 2550 6700
+F 0 "#PWR0103" H 2550 6450 50  0001 C CNN
+F 1 "GND" V 2555 6572 50  0000 R CNN
+F 2 "" H 2550 6700 50  0001 C CNN
+F 3 "" H 2550 6700 50  0001 C CNN
+	1    2550 6700
+	0    1    1    0
+$EndComp
+$Comp
+L power:GND #PWR0104
+U 1 1 61A10755
+P 2550 6800
+F 0 "#PWR0104" H 2550 6550 50  0001 C CNN
+F 1 "GND" V 2555 6672 50  0000 R CNN
+F 2 "" H 2550 6800 50  0001 C CNN
+F 3 "" H 2550 6800 50  0001 C CNN
+	1    2550 6800
+	0    1    1    0
+$EndComp
 $EndSCHEMATC

Commit message: traces ran
Parts:
- added MX41: MX-NoLED, MX_Alps_Hybrid:MX-1U-NoLED, symbol MX_Alps_Hybrid:MX-NoLED
- added MX42: MX-NoLED, MX_Alps_Hybrid:MX-7U-ReversedStabilizers-NoLED, symbol MX_Alps_Hybrid:MX-NoLED
Connections:
- net COL13 is gone; now on net COL12: MX40.1 (COL), SW1.S1
- net COL0: now also MX1.1 (COL), MX13.1 (COL), MX25.1 (COL), U1.24 (RAW)
- net COL1: now also MX14.1 (COL), MX2.1 (COL), MX26.1 (COL), U1.17 (F7); no longer MX1.1 (COL), MX13.1 (COL), MX25.1 (COL)
- net COL10: now also MX11.1 (COL), MX23.1 (COL), U1.8 (C6); no longer MX10.1 (COL), MX22.1 (COL), MX34.1 (COL)
- net COL11: now also MX12.1 (COL), MX24.1 (COL), MX35.1 (COL), MX39.1 (COL), U1.7 (D4); no longer MX11.1 (COL), MX23.1 (COL)
- net COL12: now also U1.6 (SDA), MX41.2 (ROW); no longer MX12.1 (COL), MX24.1 (COL), MX35.1 (COL), MX39.1 (COL)
- net COL2: now also MX15.1 (COL), MX27.1 (COL), MX3.1 (COL), U1.16 (B1); no longer MX14.1 (COL), MX2.1 (COL), MX26.1 (COL)
- net COL3: now also MX16.1 (COL), MX28.1 (COL), MX4.1 (COL), U1.13 (B6); no longer MX15.1 (COL), MX27.1 (COL), MX3.1 (COL)
- net COL4: now also MX17.1 (COL), MX29.1 (COL), MX5.1 (COL), U1.14 (B2); no longer MX16.1 (COL), MX28.1 (COL), MX4.1 (COL)
- net COL5: now also MX18.1 (COL), MX30.1 (COL), MX38.1 (COL), MX6.1 (COL), U1.15 (B3); no longer MX17.1 (COL), MX29.1 (COL), MX5.1 (COL)
- net COL6: now also MX19.1 (COL), MX31.1 (COL), MX7.1 (COL), U1.12 (B5); no longer MX18.1 (COL), MX30.1 (COL), MX38.1 (COL), MX6.1 (COL)
- net COL7: now also MX20.1 (COL), MX32.1 (COL), MX8.1 (COL), U1.11 (B4); no longer MX19.1 (COL), MX31.1 (COL), MX7.1 (COL)
- net COL8: now also MX21.1 (COL), MX33.1 (COL), MX9.1 (COL), U1.10 (E6); no longer MX20.1 (COL), MX32.1 (COL), MX8.1 (COL)
- net COL9: now also MX10.1 (COL), MX22.1 (COL), MX34.1 (COL), U1.9 (D7); no longer MX21.1 (COL), MX33.1 (COL), MX9.1 (COL)
- net ROW0: now also U1.1 (TX)
- net ROW1: now also U1.18 (F6)
- net ROW2: now also U1.19 (F5)
- net ROW3: now also U1.20 (F4)
- net at D13.2 (A), SW1.S2: now also MX41.1 (COL)
Other:
- moved on the sheet: D37, D38, MX36, MX37
Changed lines of the file:
@@
 L MX_Alps_Hybrid:MX-NoLED MX36
 U 1 1 61B1F48B
-P 1200 3050
-F 0 "MX36" H 1233 3273 60  0000 C CNN
-F 1 "MX-NoLED" H 1233 3199 20  0000 C CNN
-F 2 "MX_Alps_Hybrid:MX-1U-NoLED" H 575 3025 60  0001 C CNN
-F 3 "" H 575 3025 60  0001 C CNN
-	1    1200 3050
-	1    0    0    -1
-$EndComp
-$Comp
-L MX_Alps_Hybrid:MX-NoLED MX37
-U 1 1 61B1F495
 P 1700 3050
-F 0 "MX37" H 1733 3273 60  0000 C CNN
+F 0 "MX36" H 1733 3273 60  0000 C CNN
 F 1 "MX-NoLED" H 1733 3199 20  0000 C CNN
 F 2 "MX_Alps_Hybrid:MX-1U-NoLED" H 1075 3025 60  0001 C CNN
 F 3 "" H 1075 3025 60  0001 C CNN
 	1    1700 3050
+	1    0    0    -1
+$EndComp
+$Comp
+L MX_Alps_Hybrid:MX-NoLED MX37
+U 1 1 61B1F495
+P 2200 3050
+F 0 "MX37" H 2233 3273 60  0000 C CNN
+F 1 "MX-NoLED" H 2233 3199 20  0000 C CNN
+F 2 "MX_Alps_Hybrid:MX-1U-NoLED" H 1575 3025 60  0001 C CNN
+F 3 "" H 1575 3025 60  0001 C CNN
+	1    2200 3050
 	1    0    0    -1
 $EndComp
@@
 L Device:D_Small D37
 U 1 1 61B1F4DB
-P 1150 3300
-F 0 "D37" V 1196 3232 50  0000 R CNN
-F 1 "D_Small" V 1105 3232 50  0000 R CNN
-F 2 "Diode_THT:D_A-405_P7.62mm_Horizontal" V 1150 3300 50  0001 C CNN
-F 3 "~" V 1150 3300 50  0001 C CNN
-	1    1150 3300
-	0    -1   -1   0
-$EndComp
-$Comp
-L Device:D_Small D38
-U 1 1 61B1F4E5
 P 1650 3300
-F 0 "D38" V 1696 3232 50  0000 R CNN
+F 0 "D37" V 1696 3232 50  0000 R CNN
 F 1 "D_Small" V 1605 3232 50  0000 R CNN
 F 2 "Diode_THT:D_A-405_P7.62mm_Horizontal" V 1650 3300 50  0001 C CNN
@@
 	0    -1   -1   0
 $EndComp
-Connection ~ 1150 3400
-Wire Wire Line
-	1150 3400 1000 3400
-Wire Wire Line
-	1650 3400 1150 3400
-$Comp
-L Device:D_Small D13
-U 1 1 61B28A28
-P 8200 1350
-F 0 "D13" V 8246 1282 50  0000 R CNN
-F 1 "D_Small" V 8155 1282 50  0000 R CNN
-F 2 "Diode_THT:D_A-405_P7.62mm_Horizontal" V 8200 1350 50  0001 C CNN
-F 3 "~" V 8200 1350 50  0001 C CNN
-	1    8200 1350
-	0    -1   -1   0
-$EndComp
+$Comp
+L Device:D_Small D38
+U 1 1 61B1F4E5
+P 2150 3300
+F 0 "D38" V 2196 3232 50  0000 R CNN
+F 1 "D_Small" V 2105 3232 50  0000 R CNN
+F 2 "Diode_THT:D_A-405_P7.62mm_Horizontal" V 2150 3300 50  0001 C CNN
+F 3 "~" V 2150 3300 50  0001 C CNN
+	1    2150 3300
+	0    -1   -1   0
+$EndComp
+Connection ~ 1650 3400
+Wire Wire Line
+	1650 3400 1500 3400
+Wire Wire Line
+	2150 3400 1650 3400
 Connection ~ 1650 2750
 Connection ~ 2150 2750
@@
 Connection ~ 6150 2750
 Wire Wire Line
-	1650 3400 4150 3400
-Connection ~ 1650 3400
+	2150 3400 4150 3400
+Connection ~ 2150 3400
 Wire Wire Line
 	7150 3400 8000 3400
-Wire Wire Line
-	7150 3400 4150 3400
-Connection ~ 7150 3400
-Connection ~ 4150 3400
-Wire Wire Line
-	8200 1050 8250 1050
-Wire Wire Line
-	8250 1050 8250 3000
 Wire Wire Line
 	8250 3000 8200 3000
@@
 Connection ~ 2350 1700
 Wire Wire Line
-	2350 1700 2350 2350
-Wire Wire Line
 	4350 2350 4350 3000
 Connection ~ 4350 2350
-Wire Wire Line
-	1850 1050 1850 1700
 Connection ~ 1850 1700
 Wire Wire Line
 	1850 1700 1850 2350
-Connection ~ 1850 2350
-Wire Wire Line
-	1850 2350 1850 3000
-Wire Wire Line
-	1350 3000 1350 3650
 Wire Wire Line
 	1850 3000 1850 3650
-Connection ~ 1850 3000
-Wire Wire Line
-	2350 2350 2350 3650
-Connection ~ 2350 2350
+Wire Wire Line
+	2350 2350 2350 3000
 Wire Wire Line
 	2850 2350 2850 3650
@@
 Wire Wire Line
 	1000 1450 1650 1450
-Text GLabel 1350 3650 0    50   Input ~ 0
+Text GLabel 1850 3650 0    50   Input ~ 0
 COL0
-Text GLabel 1850 3650 0    50   Input ~ 0
+Text GLabel 2350 3650 0    50   Input ~ 0
 COL1
-Text GLabel 2350 3650 0    50   Input ~ 0
+Text GLabel 2850 3650 0    50   Input ~ 0
 COL2
-Text GLabel 2850 3650 0    50   Input ~ 0
+Text GLabel 3350 3650 0    50   Input ~ 0
 COL3
-Text GLabel 3350 3650 0    50   Input ~ 0
+Text GLabel 3850 3650 0    50   Input ~ 0
 COL4
-Text GLabel 3850 3650 0    50   Input ~ 0
+Text GLabel 4350 3650 0    50   Input ~ 0
 COL5
-Text GLabel 4350 3650 0    50   Input ~ 0
+Text GLabel 4850 3650 0    50   Input ~ 0
 COL6
-Text GLabel 4850 3650 0    50   Input ~ 0
+Text GLabel 5350 3650 0    50   Input ~ 0
 COL7
-Text GLabel 5350 3650 0    50   Input ~ 0
+Text GLabel 5850 3650 0    50   Input ~ 0
 COL8
-Text GLabel 5850 3650 0    50   Input ~ 0
+Text GLabel 6350 3650 0    50   Input ~ 0
 COL9
-Text GLabel 6350 3650 0    50   Input ~ 0
+Text GLabel 6850 3650 0    50   Input ~ 0
 COL10
-Text GLabel 6850 3650 0    50   Input ~ 0
+Text GLabel 7350 3650 0    50   Input ~ 0
 COL11
-Text GLabel 7350 3650 0    50   Input ~ 0
+Text GLabel 8250 3650 0    50   Input ~ 0
 COL12
-Text GLabel 8250 3650 0    50   Input ~ 0
-COL13
 Text GLabel 1000 1450 0    50   Input ~ 0
 ROW0
@@
 Text GLabel 1000 2750 0    50   Input ~ 0
 ROW2
-Text GLabel 1000 3400 0    50   Input ~ 0
+Text GLabel 1500 3400 0    50   Input ~ 0
 ROW3
 Wire Wire Line
@@
 	0    1    1    0
 $EndComp
+Wire Wire Line
+	2350 1700 2350 2350
+Wire Wire Line
+	7150 3400 4150 3400
+Connection ~ 7150 3400
+Connection ~ 4150 3400
+Connection ~ 2350 2350
+Wire Wire Line
+	2350 3000 2350 3650
+Connection ~ 2350 3000
+Wire Wire Line
+	1850 2350 1850 3000
+Connection ~ 1850 2350
+Connection ~ 1850 3000
+Text GLabel 2550 6500 0    50   Input ~ 0
+ROW0
+Text GLabel 2550 7000 0    50   Input ~ 0
+COL12
+Text GLabel 2550 7100 0    50   Input ~ 0
+COL11
+Text GLabel 2550 7200 0    50   Input ~ 0
+COL10
+Text GLabel 2550 7300 0    50   Input ~ 0
+COL9
+Text GLabel 2550 7400 0    50   Input ~ 0
+COL8
+Text GLabel 2550 7500 0    50   Input ~ 0
+COL7
+Text GLabel 2550 7600 0    50   Input ~ 0
+COL6
+Text GLabel 3950 7600 2    50   Input ~ 0
+COL3
+Text GLabel 3950 7500 2    50   Input ~ 0
+COL4
+Text GLabel 3950 7400 2    50   Input ~ 0
+COL5
+Text GLabel 3950 7300 2    50   Input ~ 0
+COL2
+Text GLabel 3950 7200 2    50   Input ~ 0
+COL1
+Text GLabel 3950 7100 2    50   Input ~ 0
+ROW1
+Text GLabel 3950 7000 2    50   Input ~ 0
+ROW2
+Text GLabel 3950 6900 2    50   Input ~ 0
+ROW3
+Text GLabel 3950 6500 2    50   Input ~ 0
+COL0
+Wire Wire Line
+	8200 1050 8250 1050
+$Comp
+L Device:D_Small D13
+U 1 1 61B28A28
+P 8200 1350
+F 0 "D13" V 8246 1282 50  0000 R CNN
+F 1 "D_Small" V 8155 1282 50  0000 R CNN
+F 2 "Diode_THT:D_A-405_P7.62mm_Horizontal" V 8200 1350 50  0001 C CNN
+F 3 "~" V 8200 1350 50  0001 C CNN
+	1    8200 1350
+	0    -1   -1   0
+$EndComp
+Wire Wire Line
+	8250 1050 8250 3000
+$Comp
+L MX_Alps_Hybrid:MX-NoLED MX41
+U 1 1 61A79EB8
+P 8400 1100
+F 0 "MX41" V 8412 1228 60  0000 L CNN
+F 1 "MX-NoLED" V 8486 1228 20  0000 L CNN
+F 2 "MX_Alps_Hybrid:MX-1U-NoLED" H 7775 1075 60  0001 C CNN
+F 3 "" H 7775 1075 60  0001 C CNN
+	1    8400 1100
+	0    1    1    0
+$EndComp
+Connection ~ 8250 1050
+Wire Wire Line
+	8450 1250 8200 1250
+Connection ~ 8200 1250
+Wire Wire Line
+	1850 1050 1850 1700
+$Comp
+L MX_Alps_Hybrid:MX-NoLED MX42
+U 1 1 61ACE0FC
+P 4200 3950
+F 0 "MX42" H 4233 4173 60  0000 C CNN
+F 1 "MX-NoLED" H 4233 4099 20  0000 C CNN
+F 2 "MX_Alps_Hybrid:MX-7U-ReversedStabilizers-NoLED" H 3575 3925 60  0001 C CNN
+F 3 "" H 3575 3925 60  0001 C CNN
+	1    4200 3950
+	1    0    0    -1
+$EndComp
 $EndSCHEMATC
